File: Hardware/Control Board/CNIX V2 Control Board/CNIX V2 Control Board.kicad_pcb (KiCad board)
At the start: 2 copper layers, 165 x 51 mm, 110 parts, among them J1 EXT, J10 LED, J11 USB_C_Receptacle, J3 Tube Out, J4 EXT, J5 I2C_ext, J6 Prog, J7 HT, J8 GND, J9 GND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

Commit message: fixed schematic
Parts:
- moved J8 2.53 mm to (225.4, 82.0), turned to -90 degrees
Other:
- board text added: "FIXED: Swapped pinheader for VDD and GND to tube board"
- board text added: "TODO: Implement low voltage current sensing via main uC to look for faults"
- board text added: "Version: 1.0"
Changed lines of the file:
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@@
 	(footprint "Connector_PinSocket_2.54mm:PinSocket_1x02_P2.54mm_Vertical"
 		(layer "B.Cu")
-		(at 227.965 81.96 90)
+		(at 225.431807 81.969316 -90)
 		(descr "Through hole straight socket strip, 1x02, 2.54mm pitch, single row (from Kicad 4.0.7), script generated")
 		(tags "Through hole socket strip THT 1x02 2.54mm single row")
 		(property "Reference" "J8"
-			(at 0 2.77 270)
+			(at 0 2.77 90)
 			(layer "B.SilkS")
 			(effects
@@
 		)
 		(property "Value" "GND"
-			(at 0 -5.31 270)
+			(at 0 -5.31 90)
 			(layer "B.Fab")
 			(effects
@@
 		)
 		(property "Datasheet" ""
-			(at 0 0 270)
+			(at 0 0 90)
 			(unlocked yes)
 			(layer "B.Fab")
@@
 		)
 		(property "Description" "Generic connector, single row, 01x02, script generated"
-			(at 0 0 270)
+			(at 0 0 90)
 			(unlocked yes)
 			(layer "B.Fab")
@@
 		(attr through_hole)
 		(fp_line
-			(start 1.33 -3.87)
-			(end -1.33 -3.87)
+			(start 1.33 1.33)
+			(end 0 1.33)
 			(stroke
 				(width 0.12)
@@
 		)
 		(fp_line
-			(start 1.33 -3.87)
-			(end 1.33 -1.27)
+			(start 1.33 0)
+			(end 1.33 1.33)
 			(stroke
 				(width 0.12)
@@
 		)
 		(fp_line
-			(start -1.33 -3.87)
+			(start 1.33 -1.27)
 			(end -1.33 -1.27)
 			(stroke
@@
 		)
 		(fp_line
-			(start 1.33 -1.27)
+			(start -1.33 -3.87)
 			(end -1.33 -1.27)
 			(stroke
@@
 		)
 		(fp_line
-			(start 1.33 0)
-			(end 1.33 1.33)
+			(start 1.33 -3.87)
+			(end 1.33 -1.27)
 			(stroke
 				(width 0.12)
@@
 		)
 		(fp_line
-			(start 1.33 1.33)
-			(end 0 1.33)
+			(start 1.33 -3.87)
+			(end -1.33 -3.87)
 			(stroke
 				(width 0.12)
@@
 		)
 		(fp_line
-			(start 1.75 -4.3)
-			(end 1.75 1.8)
+			(start -1.8 1.8)
+			(end -1.8 -4.3)
 			(stroke
 				(width 0.05)
@@
 		)
 		(fp_line
-			(start -1.8 -4.3)
-			(end 1.75 -4.3)
+			(start 1.75 1.8)
+			(end -1.8 1.8)
 			(stroke
 				(width 0.05)
@@
 		)
 		(fp_line
-			(start 1.75 1.8)
-			(end -1.8 1.8)
+			(start -1.8 -4.3)
+			(end 1.75 -4.3)
 			(stroke
 				(width 0.05)
@@
 		)
 		(fp_line
-			(start -1.8 1.8)
-			(end -1.8 -4.3)
+			(start 1.75 -4.3)
+			(end 1.75 1.8)
 			(stroke
 				(width 0.05)
@@
 		)
 		(fp_line
-			(start 1.27 -3.81)
-			(end 1.27 0.635)
+			(start -1.27 1.27)
+			(end -1.27 -3.81)
 			(stroke
 				(width 0.1)
@@
 		)
 		(fp_line
-			(start -1.27 -3.81)
-			(end 1.27 -3.81)
+			(start 0.635 1.27)
+			(end -1.27 1.27)
 			(stroke
 				(width 0.1)
@@
 		)
 		(fp_line
-			(start 0.635 1.27)
-			(end -1.27 1.27)
+			(start -1.27 -3.81)
+			(end 1.27 -3.81)
 			(stroke
 				(width 0.1)
@@
 		)
 		(fp_line
-			(start -1.27 1.27)
-			(end -1.27 -3.81)
+			(start 1.27 -3.81)
+			(end 1.27 0.635)
 			(stroke
 				(width 0.1)
@@
 		)
 		(pad "1" thru_hole rect
-			(at 0 0 90)
+			(at 0 0 270)
 			(size 1.7 1.7)
 			(drill 1)
@@
 		)
 		(pad "2" thru_hole oval
-			(at 0 -2.54 90)
+			(at 0 -2.54 270)
 			(size 1.7 1.7)
 			(drill 1)
@@
 		)
 	)
+	(gr_text "Version: 1.0"
+		(at 78.5 130.5 0)
+		(layer "F.SilkS")
+		(effects
+			(font
+				(size 1 1)
+				(thickness 0.15)
+			)
+			(justify left bottom)
+		)
+	)
 	(gr_text "High Voltage Boost Converter"
 		(at 82.424947 86.963339 0)
@@
 		)
 	)
+	(gr_text "TODO: Implement low voltage current sensing via main uC to look for faults"
+		(at 180.25 170.75 0)
+		(layer "Cmts.User")
+		(effects
+			(font
+				(size 1.5 1.5)
+				(thickness 0.3)
+				(bold yes)
+			)
+			(justify left bottom)
+		)
+	)
+	(gr_text "FIXED: Swapped pinheader for VDD and GND to tube board"
+		(at 180.25 174.5 0)
+		(layer "Cmts.User")
+		(effects
+			(font
+				(size 1.5 1.5)
+				(thickness 0.3)
+				(bold yes)
+			)
+			(justify left bottom)
+		)
+	)
 	(dimension
 		(type aligned)
@@
 	)
 	(segment
+		(start 226.8 88.25)
+		(end 226.8 84.8)
+		(width 1)
+		(layer "F.Cu")
+		(net 6)
+	)
+	(segment
 		(start 216.111051 88.5)
 		(end 216.111051 83.931051)
@@
 	)
 	(segment
-		(start 95.28605 101.096052)
-		(end 96.44605 101.096052)
-		(width 0.4)
+		(start 226.8 84.8)
+		(end 225.431807 83.431807)
+		(width 1)
 		(layer "F.Cu")
 		(net 6)
 	)
 	(segment
-		(start 226.8 88.25)
-		(end 226.8 83.125)
-		(width 1)
+		(start 95.28605 101.096052)
+		(end 96.44605 101.096052)
+		(width 0.4)
 		(layer "F.Cu")
 		(net 6)
@@
 	)
 	(segment
-		(start 226.8 83.125)
-		(end 227.965 81.96)
-		(width 1)
-		(layer "F.Cu")
-		(net 6)
-	)
-	(segment
 		(start 216.111051 95.531051)
 		(end 216.111051 88.5)
@@
 		(width 1)
 		(layer "F.Cu")
+		(net 6)
+	)
+	(segment
+		(start 225.431807 83.431807)
+		(end 225.431807 81.969316)
+		(width 1)
+		(layer "F.Cu")

Commit message: fixed output caps and routung on pcb. Version Bump to 1.1
Parts:
- removed REF** (x2): ESD-Logo_6.6x6mm_SilkScreen, Symbol:ESD-Logo_6.6x6mm_SilkScreen
- C1, C3: value 18p -> 6p
- C110: value 1u 250V -> 2u2 250V; footprint Capacitor_SMD:C_0805_2012Metric_Pad1.18x1.45mm_HandSolder -> Capacitor_SMD:C_2220_5750Metric_Pad1.97x5.40mm_HandSolder
- C111: value 1u 250V -> 100nf 250V
- L100: value 68u, 2.8A -> 33u, 4.2A
- R105: value 47k -> 60k4
- moved C111 4.38 mm to (87.2, 118.5), turned to 90 degrees
- moved C112 2.42 mm to (89.5, 118.5), turned to 90 degrees
- moved C110 2.21 mm to (86.8, 113.2)
- moved C109 0.52 mm to (83.9, 103.0)
Routing:
- net HT: track 36.5 -> 35.2 mm
Other:
- board text added: "Version: 1.1"
- board text removed: "Version: 1.0"

Commit message: added warning for tube fail
https://www.mouser.de/ProductDetail/TDK/C5750X7T2E225K250KA?qs=vG%252BtRDh6KwCR7tEmlFz%2FKw%3D%3D
exit
quit
Parts:
- moved J8 2.56 mm to (228.0, 82.0), turned to 90 degrees
Changed lines of the file:
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@@
 	(footprint "Connector_PinSocket_2.54mm:PinSocket_1x02_P2.54mm_Vertical"
 		(layer "B.Cu")
-		(at 225.431807 81.969316 -90)
+		(at 227.987222 81.970641 90)
 		(descr "Through hole straight socket strip, 1x02, 2.54mm pitch, single row (from Kicad 4.0.7), script generated")
 		(tags "Through hole socket strip THT 1x02 2.54mm single row")
@@
 		)
 		(property "Datasheet" "~"
-			(at 0 0 90)
+			(at 0 0 270)
 			(unlocked yes)
 			(layer "B.Fab")
@@
 		)
 		(property "Description" "Generic connector, single row, 01x02, script generated"
-			(at 0 0 90)
+			(at 0 0 270)
 			(unlocked yes)
 			(layer "B.Fab")
@@
 		)
 		(property "Mouser-Nr." ""
-			(at 0 0 270)
+			(at 0 0 90)
 			(unlocked yes)
 			(layer "B.Fab")
@@
 		)
 		(property "Reichelt-Nr." ""
-			(at 0 0 270)
+			(at 0 0 90)
 			(unlocked yes)
 			(layer "B.Fab")
@@
 		(attr through_hole)
 		(fp_line
-			(start 1.33 1.33)
-			(end 0 1.33)
+			(start 1.33 -3.87)
+			(end -1.33 -3.87)
 			(stroke
 				(width 0.12)
@@
 		)
 		(fp_line
-			(start 1.33 0)
-			(end 1.33 1.33)
+			(start 1.33 -3.87)
+			(end 1.33 -1.27)
 			(stroke
 				(width 0.12)
@@
 		)
 		(fp_line
-			(start 1.33 -1.27)
+			(start -1.33 -3.87)
 			(end -1.33 -1.27)
 			(stroke
@@
 		)
 		(fp_line
-			(start -1.33 -3.87)
+			(start 1.33 -1.27)
 			(end -1.33 -1.27)
 			(stroke
@@
 		)
 		(fp_line
-			(start 1.33 -3.87)
-			(end 1.33 -1.27)
+			(start 1.33 0)
+			(end 1.33 1.33)
 			(stroke
 				(width 0.12)
@@
 		)
 		(fp_line
-			(start 1.33 -3.87)
-			(end -1.33 -3.87)
+			(start 1.33 1.33)
+			(end 0 1.33)
 			(stroke
 				(width 0.12)
@@
 		)
 		(fp_line
-			(start -1.8 1.8)
-			(end -1.8 -4.3)
+			(start 1.75 -4.3)
+			(end 1.75 1.8)
 			(stroke
 				(width 0.05)
@@
 		)
 		(fp_line
-			(start 1.75 1.8)
-			(end -1.8 1.8)
+			(start -1.8 -4.3)
+			(end 1.75 -4.3)
 			(stroke
 				(width 0.05)
@@
 		)
 		(fp_line
-			(start -1.8 -4.3)
-			(end 1.75 -4.3)
+			(start 1.75 1.8)
+			(end -1.8 1.8)
 			(stroke
 				(width 0.05)
@@
 		)
 		(fp_line
-			(start 1.75 -4.3)
-			(end 1.75 1.8)
+			(start -1.8 1.8)
+			(end -1.8 -4.3)
 			(stroke
 				(width 0.05)
@@
 		)
 		(fp_line
-			(start -1.27 1.27)
-			(end -1.27 -3.81)
+			(start 1.27 -3.81)
+			(end 1.27 0.635)
 			(stroke
 				(width 0.1)
@@
 		)
 		(fp_line
-			(start 0.635 1.27)
-			(end -1.27 1.27)
+			(start -1.27 -3.81)
+			(end 1.27 -3.81)
 			(stroke
 				(width 0.1)
@@
 		)
 		(fp_line
-			(start -1.27 -3.81)
-			(end 1.27 -3.81)
+			(start 0.635 1.27)
+			(end -1.27 1.27)
 			(stroke
 				(width 0.1)
@@
 		)
 		(fp_line
-			(start 1.27 -3.81)
-			(end 1.27 0.635)
+			(start -1.27 1.27)
+			(end -1.27 -3.81)
 			(stroke
 				(width 0.1)
@@
 		)
 		(fp_text user "${REFERENCE}"
-			(at 0 -1.27 0)
+			(at -0.530684 -1.431807 0)
 			(layer "B.Fab")
 			(effects
@@
 		)
 		(pad "1" thru_hole rect
-			(at 0 0 270)
+			(at 0 0 90)
 			(size 1.7 1.7)
 			(drill 1)
@@
 		)
 		(pad "2" thru_hole oval
-			(at 0 -2.54 270)
+			(at 0 -2.54 90)
 			(size 1.7 1.7)
 			(drill 1)
@@
 	)
 	(segment
-		(start 226.8 88.25)
-		(end 226.8 84.8)
+		(start 216.111051 88.5)
+		(end 216.111051 83.931051)
 		(width 1)
 		(layer "F.Cu")
@@
 	)
 	(segment
-		(start 216.111051 88.5)
-		(end 216.111051 83.931051)
+		(start 226.8 88.25)
+		(end 226.8 85.95)
 		(width 1)
 		(layer "F.Cu")
@@
 	)
 	(segment
-		(start 226.8 84.8)
-		(end 225.431807 83.431807)
-		(width 1)
-		(layer "F.Cu")
-		(net 6)
-	)
-	(segment
 		(start 95.28605 101.096052)
 		(end 96.44605 101.096052)
@@
 	)
 	(segment
+		(start 226.8 85.95)
+		(end 228 84.75)
+		(width 1)
+		(layer "F.Cu")
+		(net 6)
+	)
+	(segment
 		(start 226.65 88.4)
 		(end 226.8 88.25)
@@
 	)
 	(segment
-		(start 225.431807 83.431807)
-		(end 225.431807 81.969316)
+		(start 228 84.75)
+		(end 227.987222 84.737222)
+		(width 1)
+		(layer "F.Cu")
+		(net 6)
+	)
+	(segment
+		(start 227.987222 84.737222)
+		(end 227.987222 81.970641)
 		(width 1)
 		(layer "F.Cu")
