File: Hardware/Control Board/CNIX V2 Control Board/CNIX V2 Control Board.kicad_sch (KiCad schematic)
At the start: 72 parts, among them J1 EXT, J10 LED, J11 USB_C_Receptacle, J3 Tube Out, J4 EXT, J5 I2C_ext, J6 Prog, J7 HT, J8 GND, J9 GND, SW1 RST, SW2 SW_Minus, SW3 SW_Menu, SW4 SW_Plus, U1 STM32G051C8T3, U2 AP7361C-33ER-13, Y1 ABS25-32.768KHZ

Commit message: redid the entire menu structure with new file structure
Parts:
- R7, R8, R9: value 4k7 -> 18k
Changed lines of the file:
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@@
 			)
 		)
-		(property "Value" "4k7"
+		(property "Value" "18k"
 			(at 138.43 150.876 90)
 			(show_name no)
@@
 			)
 		)
-		(property "Value" "4k7"
+		(property "Value" "18k"
 			(at 138.43 159.766 90)
 			(show_name no)
@@
 			)
 		)
-		(property "Value" "4k7"
+		(property "Value" "18k"
 			(at 138.43 168.656 90)
 			(show_name no)

Commit message: cleanup of project data and files
Parts:
- removed R6: 4k7, Resistor_SMD:R_0805_2012Metric_Pad1.20x1.40mm_HandSolder, symbol Device:R_Small
- added R17, R18, R19: 4k7, Resistor_SMD:R_0805_2012Metric_Pad1.20x1.40mm_HandSolder, symbol Device:R_Small
- R16: value 2k -> 4k7; Mouser Nr. 603-RC0805FR-132KL -> 603-RC0805FR-074K7P
Connections:
- net GND: now also R17.2, R18.2, R19.2
- net at D1.1 (K): now also R18.1, R19.1
- net at D3.1 (K), R16.1: now also R17.1
Other:
- note added: "Debounce ~25ms"
- moved on the sheet: D2, R15
