File: Hardware/Tube Board/CNIX V2 Tube Board/CNIX V2 Tube Board.kicad_sch (KiCad schematic)
At the start: 50 parts, among them J1 VDD, J2 GND, J3 Tube Conn, J4 LED, J5 HT, U1 SN75468, U10 IN-4_0, U11 IN-4_1, U12 IN-4_2, U13 IN-4_3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

Commit message: added warning for tube fail
https://www.mouser.de/ProductDetail/TDK/C5750X7T2E225K250KA?qs=vG%252BtRDh6KwCR7tEmlFz%2FKw%3D%3D
exit
quit
Connections:
- net GND: now also J1.1 (Pin_1); no longer J1.2 (Pin_2)
- net VDD: now also J1.2 (Pin_2); no longer J1.1 (Pin_1)
Changed lines of the file:
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@@
 	(symbol
 		(lib_id "Connector:Conn_01x02_Socket")
-		(at 274.32 45.72 0)
+		(at 274.32 48.26 0)
+		(mirror x)
 		(unit 1)
 		(exclude_from_sim no)
@@
 		(on_board yes)
 		(dnp no)
-		(fields_autoplaced yes)
 		(property "Reference" "J1"
-			(at 275.59 45.7199 0)
+			(at 275.59 48.2601 0)
 			(effects
 				(font
@@
 		)
 		(property "Value" "VDD"
-			(at 275.59 48.2599 0)
+			(at 275.59 45.7201 0)
 			(effects
 				(font
@@
 		)
 		(property "Footprint" "Connector_PinHeader_2.54mm:PinHeader_1x02_P2.54mm_Vertical"
-			(at 274.32 45.72 0)
+			(at 274.32 48.26 0)
 			(effects
 				(font
@@
 		)
 		(property "Datasheet" "~"
-			(at 274.32 45.72 0)
+			(at 274.32 48.26 0)
 			(effects
 				(font
@@
 		)
 		(property "Description" "Generic connector, single row, 01x02, script generated"
-			(at 274.32 45.72 0)
+			(at 274.32 48.26 0)
 			(effects
 				(font
@@
 		)
 		(property "Mouser URL" ""
-			(at 274.32 45.72 0)
+			(at 274.32 48.26 0)
 			(effects
 				(font
@@
 		)
 		(property "Mouser Nr." ""
-			(at 274.32 45.72 0)
+			(at 274.32 48.26 0)
 			(effects
 				(font
