File: Hardware/Tube Board/CNIX V2 Tube Board/CNIX V2 Tube Board.kicad_pcb (KiCad board)
At the start: 2 copper layers, 185 x 51 mm, 50 parts, among them J1 VDD, J2 GND, J3 Tube Conn, J4 LED, J5 HT, U1 SN75468, U10 IN-4_0, U11 IN-4_1, U12 IN-4_2, U13 IN-4_3, U14 SN75468, U2 SN75468, U3 SN75468, U4 SN75468, U5 SN75468, U6 4028, U7 4028, U8 4028, U9 4028

Commit message: cleanup of project data and files
Parts:
- moved D12 2.12 mm to (148.5, 107.1)
- moved D11 2.10 mm to (148.5, 93.5)
- moved R10 2.10 mm to (148.5, 95.7)
- moved R11 2.03 mm to (148.5, 105.0)
Routing:
- net /LED2: track 95.4 -> 98.1 mm
- net /LED1: track 106.7 -> 104.6 mm
