File: Hardware/Addon Boards/DCF77-Addon/DCF77-Addon.kicad_pcb (KiCad board)
At the start: 2 copper layers, 77 x 47.5 mm, 20 parts, among them J1 Misc-PortD, J2 Addon_Conn, J4 Misc-PortA, J5 I2C, J6 ST-Link, J8 VDD, U1 HPP845E031R1, U2 DCF77-Module

Commit message: cleanup of project data and files
Parts:
- removed REF**: KiCad-Logo2_5mm_SilkScreen, Symbol:KiCad-Logo2_5mm_SilkScreen
- removed REF**: OSHW-Logo2_7.3x6mm_SilkScreen, Symbol:OSHW-Logo2_7.3x6mm_SilkScreen
- moved D2 23.5 mm to (190.1, 62.9)
- moved R1 23.5 mm to (192.3, 62.9)
Connections:
- R1 pad 2: GND -> /A1
Routing:
- net /A1: track 24.1 -> 34.0 mm
- net GND: vias 8 -> 17
Other:
- board text added: "~{EN} Data GND 3V3"
